File: AT-MT9P.brd (EAGLE design)
At the start: 0 parts

Commit message: [add]外枠作成
Other:
- board outline added: 38 x 34 mm
Changed lines of the file:
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@@
 <setting verticaltext="up"/>
 </settings>
-<grid distance="50" unitdist="mil" unit="mil" style="lines" multiple="1" display="no" altdistance="5" altunitdist="mil" altunit="mil"/>
+<grid distance="1" unitdist="mm" unit="mm" style="lines" multiple="1" display="no" altdistance="0.1" altunitdist="mm" altunit="mm"/>
 <layers>
 <layer number="1" name="Top" color="4" fill="1" visible="yes" active="yes"/>
@@
 <board>
 <plain>
+<wire x1="-19" y1="17" x2="-19" y2="-17" width="0.1524" layer="20"/>
+<wire x1="-19" y1="-17" x2="19" y2="-17" width="0.1524" layer="20"/>
+<wire x1="-19" y1="17" x2="19" y2="17" width="0.1524" layer="20"/>
+<wire x1="19" y1="17" x2="19" y2="-17" width="0.1524" layer="20"/>
 </plain>
 <attributes>

Commit message: [add]とりあえず実装
Parts:
- added E$1: (no value), VacuumTube:NOVAL_SOCKET
- added E$2, E$3: (no value), pinhead:1X09
Changed lines of the file:
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@@
 <setting verticaltext="up"/>
 </settings>
-<grid distance="1" unitdist="mm" unit="mm" style="lines" multiple="1" display="no" altdistance="0.1" altunitdist="mm" altunit="mm"/>
+<grid distance="1" unitdist="mm" unit="mm" style="lines" multiple="1" display="yes" altdistance="0.1" altunitdist="mm" altunit="mm"/>
 <layers>
 <layer number="1" name="Top" color="4" fill="1" visible="yes" active="yes"/>
@@
 <layer number="43" name="vRestrict" color="2" fill="10" visible="yes" active="yes"/>
 <layer number="44" name="Drills" color="7" fill="1" visible="no" active="yes"/>
-<layer number="45" name="Holes" color="7" fill="1" visible="no" active="yes"/>
+<layer number="45" name="Holes" color="7" fill="1" visible="yes" active="yes"/>
 <layer number="46" name="Milling" color="3" fill="1" visible="no" active="yes"/>
 <layer number="47" name="Measures" color="7" fill="1" visible="no" active="yes"/>
@@
 <layer number="51" name="tDocu" color="7" fill="1" visible="yes" active="yes"/>
 <layer number="52" name="bDocu" color="7" fill="1" visible="yes" active="yes"/>
+<layer number="88" name="SimResults" color="9" fill="1" visible="no" active="no"/>
+<layer number="89" name="SimProbes" color="9" fill="1" visible="no" active="no"/>
+<layer number="90" name="Modules" color="5" fill="1" visible="no" active="no"/>
+<layer number="91" name="Nets" color="2" fill="1" visible="no" active="no"/>
+<layer number="92" name="Busses" color="1" fill="1" visible="no" active="no"/>
+<layer number="93" name="Pins" color="2" fill="1" visible="no" active="no"/>
+<layer number="94" name="Symbols" color="4" fill="1" visible="no" active="no"/>
+<layer number="95" name="Names" color="7" fill="1" visible="no" active="no"/>
+<layer number="96" name="Values" color="7" fill="1" visible="no" active="no"/>
+<layer number="97" name="Info" color="7" fill="1" visible="no" active="no"/>
+<layer number="98" name="Guide" color="6" fill="1" visible="no" active="no"/>
 </layers>
 <board>
@@
 <wire x1="-19" y1="17" x2="19" y2="17" width="0.1524" layer="20"/>
 <wire x1="19" y1="17" x2="19" y2="-17" width="0.1524" layer="20"/>
+<hole x="16" y="14" drill="3.2"/>
+<hole x="16" y="-14" drill="3.2"/>
+<hole x="-16" y="-14" drill="3.2"/>
+<hole x="-16" y="14" drill="3.2"/>
+<dimension x1="-16" y1="20" x2="16" y2="20" x3="0" y3="-22" textsize="1.778" layer="1" dtype="diameter"/>
+<dimension x1="-21" y1="14" x2="-21" y2="-14" x3="24" y3="0" textsize="1.778" layer="1" dtype="diameter"/>
+<dimension x1="-20" y1="17" x2="-20" y2="14" x3="29" y3="15.5" textsize="1.778" layer="1" dtype="diameter"/>
+<dimension x1="-20" y1="-14" x2="-20" y2="-17" x3="29" y3="-15.5" textsize="1.778" layer="1" dtype="diameter"/>
+<dimension x1="-16" y1="19" x2="-19" y2="19" x3="-17.5" y3="-26" textsize="1.778" layer="1" dtype="diameter"/>
+<dimension x1="19" y1="18" x2="16" y2="18" x3="17.5" y3="-26" textsize="1.778" layer="1" dtype="diameter"/>
 </plain>
 <attributes>
@@
 </autorouter>
 <elements>
+<element name="E$1" library="VacuumTube" library_urn="urn:adsk.eagle:library:8044196" package="NOVAL_SOCKET" package3d_urn="urn:adsk.eagle:package:8044357/3" value="" x="0" y="0" smashed="yes"/>
+<element name="E$2" library="pinhead" library_urn="urn:adsk.eagle:library:325" package="1X09" package3d_urn="urn:adsk.eagle:package:22483/2" value="" x="0" y="14" smashed="yes">
+<attribute name="NAME" x="-11.5062" y="15.8288" size="1.27" layer="25" ratio="10"/>
+<attribute name="VALUE" x="-11.43" y="10.825" size="1.27" layer="27"/>
+</element>
+<element name="E$3" library="pinhead" library_urn="urn:adsk.eagle:library:325" package="1X09" package3d_urn="urn:adsk.eagle:package:22483/2" value="" x="0" y="-14" smashed="yes">
+<attribute name="NAME" x="-11.5062" y="-12.1712" size="1.27" layer="25" ratio="10"/>
+<attribute name="VALUE" x="-11.43" y="-17.175" size="1.27" layer="27"/>
+</element>
 </elements>
 <signals>
@@
 </board>
 </drawing>
+<compatibility>
+<note version="8.2" severity="warning">
+Since Version 8.2, EAGLE supports online libraries. The ids
+of those online libraries will not be understood (or retained)
+with this version.
+</note>
+<note version="8.3" severity="warning">
+Since Version 8.3, EAGLE supports URNs for individual library
+assets (packages, symbols, and devices). The URNs of those assets
+will not be understood (or retained) with this version.
+</note>
+<note version="8.3" severity="warning">
+Since Version 8.3, EAGLE supports the association of 3D packages
+with devices in libraries, schematics, and board files. Those 3D
+packages will not be understood (or retained) with this version.
+</note>
+</compatibility>
 </eagle>
